File: Firefly4_hw/Firefly4.kicad_pcb (KiCad board)
At the start: 2 copper layers, 46 parts, among them Q1 LED_RGB_WS2812B, Q2 LED_RGB_WS2812B, Q3 ALS-PT19-315C, Q4 LED_RGB, Q5 LED_RGB_WS2812B, SW1 BUTTON

Commit message: pcb done  + gerber
Parts:
- moved XL7 60.5 mm to (127.0, 125.4)
- moved Q3 58.8 mm to (120.8, 125.0), turned to 270 degrees
- moved DA2 53.5 mm to (170.3, 114.5), turned to 180 degrees
- moved XL3 52.7 mm to (151.8, 111.3), turned to 180 degrees
- moved DA1 52.0 mm to (170.6, 124.8), turned to 270 degrees
- moved C18 49.7 mm to (122.6, 125.0), turned to 90 degrees
- moved R2 48.9 mm to (124.4, 125.0), turned to 90 degrees
- moved C19 45.4 mm to (126.1, 113.2), turned to 270 degrees
- moved L1 44.6 mm to (170.3, 118.5)
- moved Q4 43.5 mm to (142.3, 118.6), turned to 90 degrees
- moved C15 41.9 mm to (147.7, 123.4), turned to 180 degrees
- moved XL2 40.4 mm to (177.8, 114.7), turned to 270 degrees
- moved XL1 39.0 mm to (155.6, 111.3)
- moved R6 37.5 mm to (173.8, 121.4)
- moved R8 31.9 mm to (171.2, 111.5)
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Connections:
- DD1 pad 16: /LED_R -> /LED_B
- DD1 pad 17: /LED_G -> /LED_R
- DD1 pad 18: /LED_B -> /LED_G
Routing:
- net GND: track 0.00 -> 242.6 mm, vias 0 -> 47
- net +3.3V: track 0.00 -> 118.8 mm, vias 0 -> 2
- net +5V: track 0.00 -> 96.2 mm, vias 0 -> 4
- net Net-(C18-Pad1): track 0.00 -> 33.9 mm, vias 0 -> 2
- net Net-(DD1-Pad10): track 0.00 -> 30.2 mm, vias 0 -> 2
- net Net-(DD1-Pad12): track 0.00 -> 27.5 mm, vias 0 -> 1
- net Net-(DD1-Pad13): track 0.00 -> 26.3 mm, vias 0 -> 1
- net Net-(DD1-Pad14): track 0.00 -> 25.2 mm, vias 0 -> 1
- net /D-: track 0.00 -> 23.9 mm, vias 0 -> 1
- net /D+: track 0.00 -> 23.1 mm, vias 0 -> 1
- net /DINO: track 0.00 -> 21.8 mm, vias 0 -> 2
- net /LDO_EN: track 0.00 -> 19.9 mm, vias 0 -> 2
- net /SWDIO: track 0.00 -> 19.8 mm, vias 0 -> 1
- net /BOOST_EN: track 0.00 -> 19.0 mm, vias 0 -> 2
- net /LED_G: track 0.00 -> 18.6 mm
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- added copper zone on B.Cu, net GND
- added copper zone on F.Cu, net GND
Other:
- board outline added: 76.7 x 17.4 mm
- rule pad_to_mask_clearance: 0.2 -> 0.1
